File: homecontroller_addon_PT1000.sch (EAGLE design)
At the start: 18 parts, among them U1 OPA2188AIDGKR, U2 OPA2188AIDGKR, U3 REF3025AIDBZTG4, U4 ADS1015IDGST, X1 S2L3.50/10/90G

Commit message: lib added
Parts:
- added RV1: (no value), WE-VS:WE-VS-82550140_0805
Connections:
- net AGND: now also RV1.1
Other:
- moved on the sheet: R10, R11, R12, R7, R8, R9
Changed lines of the file:
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@@
 <layer number="48" name="Document" color="7" fill="1" visible="no" active="no"/>
 <layer number="49" name="Reference" color="7" fill="1" visible="no" active="no"/>
+<layer number="50" name="dxf" color="7" fill="1" visible="no" active="no"/>
 <layer number="51" name="tDocu" color="7" fill="1" visible="no" active="no"/>
 <layer number="52" name="bDocu" color="7" fill="1" visible="no" active="no"/>
+<layer number="53" name="tPadExt" color="7" fill="1" visible="no" active="no"/>
+<layer number="54" name="bPadExt" color="1" fill="1" visible="no" active="no"/>
 <layer number="91" name="Nets" color="2" fill="1" visible="yes" active="yes"/>
 <layer number="92" name="Busses" color="1" fill="1" visible="yes" active="yes"/>
@@
 <layer number="97" name="Info" color="7" fill="1" visible="yes" active="yes"/>
 <layer number="98" name="Guide" color="6" fill="1" visible="yes" active="yes"/>
+<layer number="250" name="Descript" color="3" fill="1" visible="no" active="no"/>
+<layer number="251" name="SMDround" color="12" fill="11" visible="no" active="no"/>
 </layers>
 <schematic xreflabel="%F%N/%S.%C%R" xrefpart="/%S.%C%R">
@@
 <part name="AGND6" library="strasys_standard" deviceset="GND2" device="" value="AGND"/>
 <part name="R12" library="Vishay_By_element14_Batch_1" deviceset="CRCW0805105KFKEA" device="" value="105K Ohms"/>
+<part name="RV1" library="WE-VS" deviceset="WE-VS" device="_0805" technology="-82550140"/>
+<part name="AGND7" library="strasys_standard" deviceset="GND2" device="" value="AGND"/>
 </parts>
 <sheets>
@@
 <text x="40.64" y="238.76" size="1.778" layer="97">0,47µF</text>
 <text x="83.82" y="228.6" size="1.778" layer="97">0,47µF oder 1µF</text>
-<text x="40.64" y="127" size="2.54" layer="97">PT1000 Circuit 1</text>
+<text x="68.58" y="132.08" size="2.54" layer="97">PT1000 Circuit 1</text>
 </plain>
 <instances>
@@
 </instance>
 <instance part="AGND5" gate="G$1" x="43.18" y="220.98"/>
-<instance part="R7" gate="A" x="73.66" y="109.22"/>
-<instance part="R8" gate="A" x="58.42" y="109.22" smashed="yes">
-<attribute name="VALUE" x="57.8358" y="103.0224" size="2.1844" layer="96" ratio="10" rot="SR0"/>
-<attribute name="NAME" x="59.4106" y="111.9886" size="2.0828" layer="95" ratio="10" rot="SR0"/>
-</instance>
-<instance part="R9" gate="A" x="27.94" y="109.22" smashed="yes">
-<attribute name="VALUE" x="27.3558" y="103.0224" size="2.1844" layer="96" ratio="10" rot="SR0"/>
-<attribute name="NAME" x="28.9306" y="111.9886" size="2.0828" layer="95" ratio="10" rot="SR0"/>
-</instance>
-<instance part="R10" gate="A" x="17.78" y="91.44" smashed="yes" rot="R90">
-<attribute name="VALUE" x="23.9776" y="90.8558" size="2.1844" layer="96" ratio="10" rot="SR90"/>
-<attribute name="NAME" x="15.0114" y="92.4306" size="2.0828" layer="95" ratio="10" rot="SR90"/>
-</instance>
-<instance part="R11" gate="A" x="48.26" y="91.44" smashed="yes" rot="R90">
-<attribute name="VALUE" x="54.4576" y="90.8558" size="2.1844" layer="96" ratio="10" rot="SR90"/>
-<attribute name="NAME" x="45.4914" y="92.4306" size="2.0828" layer="95" ratio="10" rot="SR90"/>
-</instance>
-<instance part="AGND6" gate="G$1" x="48.26" y="83.82"/>
-<instance part="R12" gate="A" x="81.28" y="93.98" smashed="yes">
-<attribute name="VALUE" x="80.6958" y="87.7824" size="2.1844" layer="96" ratio="10" rot="SR0"/>
-<attribute name="NAME" x="82.2706" y="96.7486" size="2.0828" layer="95" ratio="10" rot="SR0"/>
-</instance>
+<instance part="R7" gate="A" x="101.6" y="114.3"/>
+<instance part="R8" gate="A" x="86.36" y="114.3" smashed="yes">
+<attribute name="VALUE" x="85.7758" y="108.1024" size="2.1844" layer="96" ratio="10" rot="SR0"/>
+<attribute name="NAME" x="87.3506" y="117.0686" size="2.0828" layer="95" ratio="10" rot="SR0"/>
+</instance>
+<instance part="R9" gate="A" x="55.88" y="114.3" smashed="yes">
+<attribute name="VALUE" x="55.2958" y="108.1024" size="2.1844" layer="96" ratio="10" rot="SR0"/>
+<attribute name="NAME" x="56.8706" y="117.0686" size="2.0828" layer="95" ratio="10" rot="SR0"/>
+</instance>
+<instance part="R10" gate="A" x="45.72" y="96.52" smashed="yes" rot="R90">
+<attribute name="VALUE" x="51.9176" y="95.9358" size="2.1844" layer="96" ratio="10" rot="SR90"/>
+<attribute name="NAME" x="42.9514" y="97.5106" size="2.0828" layer="95" ratio="10" rot="SR90"/>
+</instance>
+<instance part="R11" gate="A" x="76.2" y="96.52" smashed="yes" rot="R90">
+<attribute name="VALUE" x="82.3976" y="95.9358" size="2.1844" layer="96" ratio="10" rot="SR90"/>
+<attribute name="NAME" x="73.4314" y="97.5106" size="2.0828" layer="95" ratio="10" rot="SR90"/>
+</instance>
+<instance part="AGND6" gate="G$1" x="76.2" y="88.9"/>
+<instance part="R12" gate="A" x="109.22" y="99.06" smashed="yes">
+<attribute name="VALUE" x="108.6358" y="92.8624" size="2.1844" layer="96" ratio="10" rot="SR0"/>
+<attribute name="NAME" x="110.2106" y="101.8286" size="2.0828" layer="95" ratio="10" rot="SR0"/>
+</instance>
+<instance part="RV1" gate="G$1" x="20.32" y="83.82" rot="R90"/>
+<instance part="AGND7" gate="G$1" x="20.32" y="73.66"/>
 </instances>
 <busses>
@@
 <segment>
 <pinref part="R11" gate="A" pin="2"/>
-<wire x1="48.26" y1="91.44" x2="48.26" y2="86.36" width="0.1524" layer="91"/>
+<wire x1="76.2" y1="96.52" x2="76.2" y2="91.44" width="0.1524" layer="91"/>
 <pinref part="AGND6" gate="G$1" pin="GND2"/>
+</segment>
+<segment>
+<pinref part="AGND7" gate="G$1" pin="GND2"/>
+<pinref part="RV1" gate="G$1" pin="1"/>
+<wire x1="20.32" y1="76.2" x2="20.32" y2="78.74" width="0.1524" layer="91"/>
 </segment>
 </net>
@@
 </segment>
 <segment>
-<wire x1="83.82" y1="119.38" x2="83.82" y2="116.84" width="0.1524" layer="91"/>
+<wire x1="111.76" y1="124.46" x2="111.76" y2="121.92" width="0.1524" layer="91"/>
 <pinref part="R7" gate="A" pin="2"/>
-<label x="106.68" y="104.14" size="1.778" layer="95"/>
+<label x="134.62" y="109.22" size="1.778" layer="95"/>
 <pinref part="R12" gate="A" pin="1"/>
-<wire x1="93.98" y1="93.98" x2="101.6" y2="93.98" width="0.1524" layer="91"/>
-<wire x1="101.6" y1="93.98" x2="101.6" y2="104.14" width="0.1524" layer="91"/>
-<wire x1="101.6" y1="104.14" x2="101.6" y2="119.38" width="0.1524" layer="91"/>
-<wire x1="101.6" y1="119.38" x2="83.82" y2="119.38" width="0.1524" layer="91"/>
-<wire x1="106.68" y1="104.14" x2="101.6" y2="104.14" width="0.1524" layer="91"/>
-<junction x="101.6" y="104.14"/>
+<wire x1="121.92" y1="99.06" x2="129.54" y2="99.06" width="0.1524" layer="91"/>
+<wire x1="129.54" y1="99.06" x2="129.54" y2="109.22" width="0.1524" layer="91"/>
+<wire x1="129.54" y1="109.22" x2="129.54" y2="124.46" width="0.1524" layer="91"/>
+<wire x1="129.54" y1="124.46" x2="111.76" y2="124.46" width="0.1524" layer="91"/>
+<wire x1="134.62" y1="109.22" x2="129.54" y2="109.22" width="0.1524" layer="91"/>
+<junction x="129.54" y="109.22"/>
 </segment>
 </net>
@@
 </segment>
 <segment>
-<wire x1="17.78" y1="114.3" x2="17.78" y2="109.22" width="0.1524" layer="91"/>
-<wire x1="17.78" y1="104.14" x2="17.78" y2="109.22" width="0.1524" layer="91"/>
+<wire x1="45.72" y1="119.38" x2="45.72" y2="114.3" width="0.1524" layer="91"/>
+<wire x1="45.72" y1="109.22" x2="45.72" y2="114.3" width="0.1524" layer="91"/>
 <pinref part="R9" gate="A" pin="2"/>
-<wire x1="27.94" y1="109.22" x2="17.78" y2="109.22" width="0.1524" layer="91"/>
-<junction x="17.78" y="109.22"/>
+<wire x1="55.88" y1="114.3" x2="45.72" y2="114.3" width="0.1524" layer="91"/>
+<junction x="45.72" y="114.3"/>
 <pinref part="R10" gate="A" pin="1"/>
-<label x="22.86" y="116.84" size="1.778" layer="95" rot="R180"/>
+<label x="50.8" y="121.92" size="1.778" layer="95" rot="R180"/>
 </segment>
 </net>
@@
 <segment>
 <pinref part="R10" gate="A" pin="2"/>
-<wire x1="17.78" y1="91.44" x2="17.78" y2="83.82" width="0.1524" layer="91"/>
-<label x="25.4" y="83.82" size="1.778" layer="95" rot="R180"/>
+<wire x1="45.72" y1="96.52" x2="45.72" y2="88.9" width="0.1524" layer="91"/>
+<label x="53.34" y="88.9" size="1.778" layer="95" rot="R180"/>
 </segment>
 </net>
@@
 <net name="N$2" class="0">
 <segment>
-<wire x1="48.26" y1="104.14" x2="48.26" y2="109.22" width="0.1524" layer="91"/>
-<wire x1="48.26" y1="109.22" x2="58.42" y2="109.22" width="0.1524" layer="91"/>
+<wire x1="76.2" y1="109.22" x2="76.2" y2="114.3" width="0.1524" layer="91"/>
+<wire x1="76.2" y1="114.3" x2="86.36" y2="114.3" width="0.1524" layer="91"/>
 <pinref part="R8" gate="A" pin="2"/>
 <pinref part="R9" gate="A" pin="1"/>
-<wire x1="48.26" y1="109.22" x2="40.64" y2="109.22" width="0.1524" layer="91"/>
-<junction x="48.26" y="109.22"/>
+<wire x1="76.2" y1="114.3" x2="68.58" y2="114.3" width="0.1524" layer="91"/>
+<junction x="76.2" y="114.3"/>
 <pinref part="R11" gate="A" pin="1"/>
 </segment>
@@
 <pinref part="R7" gate="A" pin="1"/>
 <pinref part="R8" gate="A" pin="1"/>
-<wire x1="73.66" y1="109.22" x2="71.12" y2="109.22" width="0.1524" layer="91"/>
+<wire x1="101.6" y1="114.3" x2="99.06" y2="114.3" width="0.1524" layer="91"/>
 </segment>
 </net>
@@
 <segment>
 <pinref part="R12" gate="A" pin="2"/>
-<wire x1="81.28" y1="93.98" x2="73.66" y2="93.98" width="0.1524" layer="91"/>
-<label x="66.04" y="93.98" size="1.778" layer="95"/>
-</segment>
-<segment>
+<wire x1="109.22" y1="99.06" x2="101.6" y2="99.06" width="0.1524" layer="91"/>
+<label x="93.98" y="99.06" size="1.778" layer="95"/>
+</segment>
+<segment>

Commit message: update lib
Parts:
- added C1: 1000pF, supply2:C1206C102KDRACTU
- added C2, C3: 0.1uF, Kemet_By_element14_1:C0805F104K5RACAUTO
Connections:
- removed net N$2: R11.1, R8.2, R9.1
- new net -IN_1: R11.1, R8.2, R9.1, U1.-IN_B
- net AGND: now also C1.C1, C2.C1, C3.C1
- net PT1000_1: now also C1.C2, RV1.2
- net REF2.0V: now also C3.C2
- net VDD5V_F: now also C2.C2
Other:
- note removed: "0,47µF oder 1µF"
- moved on the sheet: R11, RV1
Changed lines of the file:
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@@
 <part name="RV1" library="WE-VS" deviceset="WE-VS" device="_0805" technology="-82550140"/>
 <part name="AGND7" library="strasys_standard" deviceset="GND2" device="" value="AGND"/>
+<part name="C1" library="supply2" deviceset="C1206C102KDRACTU" device="" value="1000pF"/>
+<part name="AGND8" library="strasys_standard" deviceset="GND2" device="" value="AGND"/>
+<part name="C2" library="Kemet_By_element14_1" deviceset="C0805F104K5RACAUTO" device="" value="0.1uF"/>
+<part name="AGND9" library="strasys_standard" deviceset="GND2" device="" value="AGND"/>
+<part name="C3" library="Kemet_By_element14_1" deviceset="C0805F104K5RACAUTO" device="" value="0.1uF"/>
+<part name="AGND10" library="strasys_standard" deviceset="GND2" device="" value="AGND"/>
 </parts>
 <sheets>
@@
 <text x="259.08" y="116.84" size="1.778" layer="97">0-4.096 V (= full scale)</text>
 <text x="40.64" y="238.76" size="1.778" layer="97">0,47µF</text>
-<text x="83.82" y="228.6" size="1.778" layer="97">0,47µF oder 1µF</text>
 <text x="68.58" y="132.08" size="2.54" layer="97">PT1000 Circuit 1</text>
 </plain>
@@
 <attribute name="NAME" x="188.9506" y="157.7086" size="2.0828" layer="95" ratio="10" rot="SR0"/>
 </instance>
-<instance part="AGND5" gate="G$1" x="43.18" y="220.98"/>
+<instance part="AGND5" gate="G$1" x="48.26" y="220.98"/>
 <instance part="R7" gate="A" x="101.6" y="114.3"/>
 <instance part="R8" gate="A" x="86.36" y="114.3" smashed="yes">
@@
 <attribute name="NAME" x="42.9514" y="97.5106" size="2.0828" layer="95" ratio="10" rot="SR90"/>
 </instance>
-<instance part="R11" gate="A" x="76.2" y="96.52" smashed="yes" rot="R90">
-<attribute name="VALUE" x="82.3976" y="95.9358" size="2.1844" layer="96" ratio="10" rot="SR90"/>
-<attribute name="NAME" x="73.4314" y="97.5106" size="2.0828" layer="95" ratio="10" rot="SR90"/>
-</instance>
-<instance part="AGND6" gate="G$1" x="76.2" y="88.9"/>
+<instance part="R11" gate="A" x="76.2" y="78.74" smashed="yes" rot="R90">
+<attribute name="VALUE" x="82.3976" y="78.1558" size="2.1844" layer="96" ratio="10" rot="SR90"/>
+<attribute name="NAME" x="73.4314" y="82.2706" size="2.0828" layer="95" ratio="10" rot="SR90"/>
+</instance>
+<instance part="AGND6" gate="G$1" x="76.2" y="73.66"/>
 <instance part="R12" gate="A" x="109.22" y="99.06" smashed="yes">
 <attribute name="VALUE" x="108.6358" y="92.8624" size="2.1844" layer="96" ratio="10" rot="SR0"/>
 <attribute name="NAME" x="110.2106" y="101.8286" size="2.0828" layer="95" ratio="10" rot="SR0"/>
 </instance>
-<instance part="RV1" gate="G$1" x="20.32" y="83.82" rot="R90"/>
-<instance part="AGND7" gate="G$1" x="20.32" y="73.66"/>
+<instance part="RV1" gate="G$1" x="35.56" y="83.82" rot="R90"/>
+<instance part="AGND7" gate="G$1" x="35.56" y="73.66"/>
+<instance part="C1" gate="G$1" x="45.72" y="81.28" smashed="yes" rot="R90">
+<attribute name="VALUE" x="49.9872" y="78.1558" size="2.1844" layer="96" ratio="10" rot="SR90"/>
+<attribute name="NAME" x="42.9514" y="80.3656" size="2.0828" layer="95" ratio="10" rot="SR90"/>
+</instance>
+<instance part="AGND8" gate="G$1" x="45.72" y="73.66"/>
+<instance part="C2" gate="A" x="33.02" y="226.06" smashed="yes" rot="R90">
+<attribute name="VALUE" x="39.8272" y="225.4758" size="2.1844" layer="96" ratio="10" rot="SR90"/>
+<attribute name="NAME" x="30.2514" y="225.1456" size="2.0828" layer="95" ratio="10" rot="SR90"/>
+</instance>
+<instance part="AGND9" gate="G$1" x="33.02" y="220.98"/>
+<instance part="C3" gate="A" x="93.98" y="226.06" smashed="yes" rot="R90">
+<attribute name="VALUE" x="100.7872" y="225.4758" size="2.1844" layer="96" ratio="10" rot="SR90"/>
+<attribute name="NAME" x="91.2114" y="225.1456" size="2.0828" layer="95" ratio="10" rot="SR90"/>
+</instance>
+<instance part="AGND10" gate="G$1" x="93.98" y="220.98"/>
 </instances>
 <busses>
@@
 <pinref part="U3" gate="A" pin="GND"/>
 <pinref part="AGND5" gate="G$1" pin="GND2"/>
-<wire x1="50.8" y1="228.6" x2="43.18" y2="228.6" width="0.1524" layer="91"/>
-<wire x1="43.18" y1="228.6" x2="43.18" y2="223.52" width="0.1524" layer="91"/>
+<wire x1="50.8" y1="228.6" x2="48.26" y2="228.6" width="0.1524" layer="91"/>
+<wire x1="48.26" y1="228.6" x2="48.26" y2="223.52" width="0.1524" layer="91"/>
 </segment>
 <segment>
 <pinref part="R11" gate="A" pin="2"/>
-<wire x1="76.2" y1="96.52" x2="76.2" y2="91.44" width="0.1524" layer="91"/>
+<wire x1="76.2" y1="78.74" x2="76.2" y2="76.2" width="0.1524" layer="91"/>
 <pinref part="AGND6" gate="G$1" pin="GND2"/>
 </segment>
@@
 <pinref part="AGND7" gate="G$1" pin="GND2"/>
 <pinref part="RV1" gate="G$1" pin="1"/>
-<wire x1="20.32" y1="76.2" x2="20.32" y2="78.74" width="0.1524" layer="91"/>
+<wire x1="35.56" y1="76.2" x2="35.56" y2="78.74" width="0.1524" layer="91"/>
+</segment>
+<segment>
+<pinref part="C1" gate="G$1" pin="C1"/>
+<pinref part="AGND8" gate="G$1" pin="GND2"/>
+<wire x1="45.72" y1="81.28" x2="45.72" y2="76.2" width="0.1524" layer="91"/>
+</segment>
+<segment>
+<pinref part="C2" gate="A" pin="C1"/>
+<pinref part="AGND9" gate="G$1" pin="GND2"/>
+<wire x1="33.02" y1="226.06" x2="33.02" y2="223.52" width="0.1524" layer="91"/>
+</segment>
+<segment>
+<pinref part="C3" gate="A" pin="C1"/>
+<pinref part="AGND10" gate="G$1" pin="GND2"/>
+<wire x1="93.98" y1="226.06" x2="93.98" y2="223.52" width="0.1524" layer="91"/>
 </segment>
 </net>
@@
 <segment>
 <pinref part="U3" gate="A" pin="IN"/>
-<wire x1="50.8" y1="233.68" x2="40.64" y2="233.68" width="0.1524" layer="91"/>
-<label x="27.94" y="233.68" size="1.778" layer="95"/>
+<wire x1="50.8" y1="233.68" x2="33.02" y2="233.68" width="0.1524" layer="91"/>
+<label x="15.24" y="233.68" size="1.778" layer="95"/>
+<pinref part="C2" gate="A" pin="C2"/>
+<wire x1="33.02" y1="233.68" x2="25.4" y2="233.68" width="0.1524" layer="91"/>
+<junction x="33.02" y="233.68"/>
 </segment>
 <segment>
@@
 <segment>
 <pinref part="U3" gate="A" pin="OUT"/>
-<wire x1="86.36" y1="233.68" x2="101.6" y2="233.68" width="0.1524" layer="91"/>
+<wire x1="86.36" y1="233.68" x2="93.98" y2="233.68" width="0.1524" layer="91"/>
 <label x="104.14" y="233.68" size="1.778" layer="95"/>
+<wire x1="93.98" y1="233.68" x2="101.6" y2="233.68" width="0.1524" layer="91"/>
 <wire x1="101.6" y1="233.68" x2="101.6" y2="215.9" width="0.1524" layer="91"/>
 <pinref part="R2" gate="A" pin="1"/>
@@
 <wire x1="111.76" y1="215.9" x2="101.6" y2="215.9" width="0.1524" layer="91"/>
 <junction x="101.6" y="215.9"/>
+<pinref part="C3" gate="A" pin="C2"/>
+<junction x="93.98" y="233.68"/>
 </segment>
 <segment>
@@
 <pinref part="R10" gate="A" pin="2"/>
 <wire x1="45.72" y1="96.52" x2="45.72" y2="88.9" width="0.1524" layer="91"/>
-<label x="53.34" y="88.9" size="1.778" layer="95" rot="R180"/>
+<pinref part="RV1" gate="G$1" pin="2"/>
+<wire x1="45.72" y1="91.44" x2="35.56" y2="91.44" width="0.1524" layer="91"/>
+<wire x1="35.56" y1="91.44" x2="27.94" y2="91.44" width="0.1524" layer="91"/>
+<wire x1="35.56" y1="88.9" x2="35.56" y2="91.44" width="0.1524" layer="91"/>
+<pinref part="C1" gate="G$1" pin="C2"/>
+<wire x1="45.72" y1="88.9" x2="45.72" y2="91.44" width="0.1524" layer="91"/>
+<junction x="35.56" y="91.44"/>
+<junction x="45.72" y="91.44"/>
+<label x="22.86" y="93.98" size="1.778" layer="95"/>
 </segment>
 </net>
@@
 </segment>
 </net>
-<net name="N$2" class="0">
-<segment>
-<wire x1="76.2" y1="109.22" x2="76.2" y2="114.3" width="0.1524" layer="91"/>
+<net name="-IN_1" class="0">
+<segment>
+<wire x1="76.2" y1="91.44" x2="76.2" y2="99.06" width="0.1524" layer="91"/>
+<wire x1="76.2" y1="99.06" x2="76.2" y2="114.3" width="0.1524" layer="91"/>
 <wire x1="76.2" y1="114.3" x2="86.36" y2="114.3" width="0.1524" layer="91"/>
 <pinref part="R8" gate="A" pin="2"/>
@@
 <junction x="76.2" y="114.3"/>
 <pinref part="R11" gate="A" pin="1"/>
+<wire x1="76.2" y1="99.06" x2="83.82" y2="99.06" width="0.1524" layer="91"/>
+<junction x="76.2" y="99.06"/>
+<label x="81.28" y="101.6" size="1.778" layer="95"/>
+</segment>
+<segment>
+<pinref part="U1" gate="A" pin="-IN_B"/>
+<wire x1="175.26" y1="177.8" x2="172.72" y2="177.8" width="0.1524" layer="91"/>
+<label x="165.1" y="177.8" size="1.778" layer="95"/>
 </segment>
 </net>
@@
 <pinref part="R12" gate="A" pin="2"/>
 <wire x1="109.22" y1="99.06" x2="101.6" y2="99.06" width="0.1524" layer="91"/>
-<label x="93.98" y="99.06" size="1.778" layer="95"/>
-</segment>
-<segment>
+<label x="99.06" y="101.6" size="1.778" layer="95"/>
+</segment>
+<segment>

Commit message: finalised sch
Parts:
- added C4, C8, C9: 1000pF, supply2:C1206C102KDRACTU
- added C5, C6, C7: 0.1uF, Kemet_By_element14_1:C0805F104K5RACAUTO
- added R13: 10K Ohms, Vishay_By_element14_Batch_1:CRCW080510K0JNEA
- added R14, R20: 10KOHM, Panasonic-Trimmer_Potentiometers:EVM3YSX50B14-3W
- added R15, R21: 30K Ohms, Vishay_By_element14_Batch_1:CRCW080530K0FKEA
- added R16, R22: 32.4K Ohms, Vishay_By_element14_Batch_1:CRCW080532K4FKEA
- added R17, R23: 24.9K Ohms, Vishay_By_element14_Batch_1:CRCW080524K9FKEA
- added R18, R24: 1K Ohm, Vishay_By_element14_Batch_1:CRCW08051K00FKTC
- added R19, R25: 105K Ohms, Vishay_By_element14_Batch_1:CRCW0805105KFKEA
- added RV2, RV3, RV4: (no value), WE-VS:WE-VS-82550140_0805
Connections:
- new net +IN_2: R19.2, U2.+IN_A
- new net +IN_3: R25.2, U2.+IN_B
- new net -IN_2: R15.2, R16.1, R18.1, U2.-IN_A
- new net -IN_3: R21.2, R22.1, R24.1, U2.-IN_B
- new net N$2: R14.1, R15.1
- new net N$4: R20.1, R21.1
- net +3.3V: now also R13.1
- net AGND: now also C4.C1, C5.C2, C6.C2, C7.C2, C8.C1, C9.C1, R18.2, R24.2, RV2.1, RV3.1, RV4.1, U2.V-
- net AIN2: now also R14.2, R19.1
- net AIN3: now also R20.2, R25.1
- net P9_14: now also R13.2, U4.ALERT/RDY
- net PT1000_0: now also C4.C2, RV2.2
- net PT1000_2: now also C8.C2, R17.2, RV3.2
- net PT1000_3: now also C9.C2, R23.2, RV4.2
- net REF2.0V: now also R16.2, R17.1, R22.2, R23.1
- net VDD5V_F: now also C5.C1, C6.C1, C7.C1, U2.V+
Other:
- note added: "PT1000 Circuit 2"
- note added: "PT1000 Circuit 3"
- note removed: "0,47µF"
- moved on the sheet: X2
