File: homecontroller_addon_PT1000.brd (EAGLE design)
At the start: 60 x 100 mm, 48 parts, among them U1 OPA2188AIDGKR, U2 OPA2188AIDGKR, U3 REF3025AIDBZTG4, U4 ADS1015IDGST, X1 S2L3.50/10/90G

Commit message: update PT1000
Parts:
- added R27, R28: 4.7K Ohms, Vishay_By_element14_Batch_1:RESC2013X65N
Connections:
- net +3.3V: now also R27.1, R28.1
- net I2C1_SCL: now also R28.2
- net I2C1_SDA: now also R27.2
Routing:
- net I2C1_SDA: track 60.9 -> 65.6 mm
- net I2C1_SCL: track 57.2 -> 60.7 mm
- net +3.3V: track 102.5 -> 105.3 mm, vias 1 -> 2
Changed lines of the file:
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@@
 <attribute name="MPN" value="" x="21.1" y="5.4" size="1.778" layer="27" rot="R180" display="off"/>
+</element>
+<element name="R27" library="Vishay_By_element14_Batch_1" package="RESC2013X65N" value="4.7K Ohms" x="13.1" y="2.5" smashed="yes" rot="R180">
+<attribute name="OC_NEWARK" value="53K0215" x="13.1" y="2.5" size="1.778" layer="27" rot="R180" display="off"/>
+<attribute name="TOLERANCE" value="±1%" x="13.1" y="2.5" size="1.778" layer="27" rot="R180" display="off"/>
+<attribute name="MPN" value="CRCW08054K70FKEA" x="13.1" y="2.5" size="1.778" layer="27" rot="R180" display="off"/>
+<attribute name="SUPPLIER" value="Vishay" x="13.1" y="2.5" size="1.778" layer="27" rot="R180" display="off"/>
+<attribute name="OC_FARNELL" value="1469923" x="13.1" y="2.5" size="1.778" layer="27" rot="R180" display="off"/>
+<attribute name="WATTAGE" value="0.125 W" x="13.1" y="2.5" size="1.778" layer="27" rot="R180" display="off"/>
+<attribute name="NAME" x="8.4456" y="2.17" size="1" layer="25" rot="SR0"/>
+<attribute name="VALUE" x="16.5544" y="5.675" size="2.0828" layer="27" ratio="10" rot="SR180"/>
+</element>
+<element name="R28" library="Vishay_By_element14_Batch_1" package="RESC2013X65N" value="4.7K Ohms" x="17.7" y="2.5" smashed="yes">
+<attribute name="OC_NEWARK" value="53K0215" x="17.7" y="2.5" size="1.778" layer="27" display="off"/>
+<attribute name="TOLERANCE" value="±1%" x="17.7" y="2.5" size="1.778" layer="27" display="off"/>
+<attribute name="MPN" value="CRCW08054K70FKEA" x="17.7" y="2.5" size="1.778" layer="27" display="off"/>
+<attribute name="SUPPLIER" value="Vishay" x="17.7" y="2.5" size="1.778" layer="27" display="off"/>
+<attribute name="OC_FARNELL" value="1469923" x="17.7" y="2.5" size="1.778" layer="27" display="off"/>
+<attribute name="WATTAGE" value="0.125 W" x="17.7" y="2.5" size="1.778" layer="27" display="off"/>
+<attribute name="NAME" x="20.0456" y="1.97" size="1" layer="25" rot="SR0"/>
+<attribute name="VALUE" x="14.2456" y="-0.675" size="2.0828" layer="27" ratio="10" rot="SR0"/>
 </element>
 </elements>
@@
 <via x="16" y="53.6" extent="1-16" drill="0.3"/>
 <wire x1="16" y1="53.6" x2="16" y2="55.9302" width="0.15" layer="1"/>
+<contactref element="R28" pad="1"/>
+<contactref element="R27" pad="1"/>
+<via x="15.4" y="2.5" extent="1-16" drill="0.3"/>
+<wire x1="14.0398" y1="2.5" x2="15.4" y2="2.5" width="0.15" layer="1"/>
+<wire x1="16.7602" y1="2.5" x2="16.7602" y2="2.5602" width="0.15" layer="1"/>
+<wire x1="16.7602" y1="2.5602" x2="16.8" y2="2.6" width="0.15" layer="1"/>
+<wire x1="15.4" y1="2.5" x2="16.7602" y2="2.5" width="0.15" layer="1"/>
+<wire x1="25" y1="2.6" x2="16.8" y2="2.6" width="0" layer="19" extent="1-15"/>
 </signal>
 <signal name="P9_14">
@@
 <wire x1="9.4" y1="58.2" x2="8.225" y2="58.2" width="0.15" layer="1"/>
 <wire x1="8.225" y1="58.2" x2="8.2156" y2="58.2094" width="0.15" layer="1"/>
+<contactref element="R28" pad="2"/>
+<wire x1="17.1" y1="5.4" x2="17.1" y2="4.0398" width="0.15" layer="1"/>
+<wire x1="17.1" y1="4.0398" x2="18.6398" y2="2.5" width="0.15" layer="1"/>
 </signal>
 <signal name="VDD5V_F">
@@
 <wire x1="7.7" y1="56.8" x2="7.2" y2="57.2" width="0.15" layer="1"/>
 <wire x1="7.2" y1="57.2" x2="7.2" y2="58.5" width="0.15" layer="1"/>
+<contactref element="R27" pad="2"/>
+<wire x1="15.1" y1="5.4" x2="15.1" y2="4.7" width="0.15" layer="1"/>
+<wire x1="15.1" y1="4.7" x2="14.5" y2="4.1" width="0.15" layer="1"/>
+<wire x1="14.5" y1="4.1" x2="13.4602" y2="4.1" width="0.15" layer="1"/>
+<wire x1="13.4602" y1="4.1" x2="12.1602" y2="2.5" width="0.15" layer="1"/>
 </signal>
 <signal name="N$3">
