File: EL-100-020-005-indicator-light.sch (EAGLE design)
At the start: 9 parts, among them X1 140-08-FLACHBAND1.27

Commit message: prototype order status
Parts:
- LED4: value KP-1608QBC-D-LED -> P-1608SURCK; MPC (none) -> KP-1608SURCK; OC_FARNELL (none) -> 2290329
Changed lines of the file:
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@@
 <part name="LED2" library="strasys_standard" deviceset="KP-1608QBC-D-LED" device=""/>
 <part name="LED3" library="strasys_standard" deviceset="KP-1608QBC-D-LED" device=""/>
-<part name="LED4" library="strasys_standard" deviceset="KP-1608QBC-D-LED" device=""/>
+<part name="LED4" library="strasys_standard" deviceset="KP-1608QBC-D-LED" device="" value="P-1608SURCK">
+<attribute name="MPC" value="KP-1608SURCK"/>
+<attribute name="OC_FARNELL" value="2290329"/>
+</part>
 <part name="R1" library="Vishay_By_element14_Batch_1" deviceset="CRCW08051K00JNEA" device="" value="1K Ohms"/>
 <part name="R2" library="Vishay_By_element14_Batch_1" deviceset="CRCW08051K00JNEA" device="" value="1K Ohms"/>
