File: EL-100-020-010-AnalogIN.sch (EAGLE design)
At the start: 23 parts, among them U16 24AA256-I/SN, U17 SW-DIL-3, U6 OPA2170AID

Commit message: prototype order status
Parts:
- removed C37, C38: 82000pF, Kemet_By_element14_Batch_1:C0603C823K5RACTU
- removed C39, C40: 180pF, Kemet_By_element14_Batch_1:C0603C181J2GACTU
- removed C41, C48: 0.1uF, Kemet_By_element14_Batch_1:C0603C104K5RAC-TU
- removed R56, R57, R58, R59, R82, R84, R85: 4.7K Ohms, Vishay_By_element14_Batch_1:CRCW06034K70FKEA
- removed R60, R62: 590 Ohms, Vishay_By_element14_Batch_1:CRCW0603590RFKEA
- removed R61, R63: 536 Ohms, Vishay_By_element14_Batch_1:CRCW0603536RFKEA
- removed R64, R65: 49.9 Ohms, Vishay_By_element14_Batch_1:CRCW060349R9FKEA
- removed R83: 10K Ohms, Vishay_By_element14_Batch_1:CRCW060310K0FKEA
- removed U17: SW-DIL-3, strasys_standard:SW-DIL-3
- added C1, C2, C6, C7: 0.082µF, Kemet_By_element14_1:C0805C180J5GACTU
- added C10, C4, C5, C9: 180pF, Kemet_By_element14_1:C0805C180J5GACTU
- added C12, C3, C8: 100nF, Kemet_By_element14_1:C0805C104K5RACTU
- added R1, R11, R12, R2: 9.76K Ohms, Vishay_By_element14_Batch_1:CRCW08059K76FKEA
- added R10, R17, R18, R19, R20, R7, R8, R9: 499 Ohms, Vishay_By_element14_Batch_1:CRCW0805499RFKEA
- added R13, R14, R3, R4: 5.49K Ohms, Vishay_By_element14_Batch_1:CRCW08055K49FKEA
- added R15, R16, R5, R6: 49.9 Ohms, Vishay_By_element14_Batch_1:CRCW080549R9FKEA
- added R28, R29, R30, R31, R32, R33: 10K Ohms, Vishay_By_element14_Batch_1:CRCW080510K0JNEA
- added U1: OPA2170AID, strasys_standard:OPA2170AID
- added X1: 9012-26, con-WuP:9012-26
- added X2: 944-12-08-00, strasys_standard:944-12-08-00
Connections:
- removed net 24AA_A0: R85.2, U16.A0, U17.3
- removed net DGND: C48.C1, U16.VSS, U17.4, U17.5, U17.6
- removed net N$19: R82.2, U16.A2
- removed net VDD5V_F: C41.C2, U6.V+
- new net 24AA-A0: R31.2, U16.A0, X2.2
- new net 24AA_A2: R33.2, U16.A2, X2.6
- new net AIN0: C4.C2, R7.2, R8.1, X1.A7
- new net AIN1: C5.C2, R10.1, R9.2, X1.B7
- new net AIN3_0-10V: R11.2, X1.A2
- new net AIN4_0-10V: R12.2, X1.B2
- new net N$1: C6.C2, R11.1, R13.2, U1.+IN_A
- new net N$3: C7.C2, R12.1, R14.2, U1.+IN_B
- new net OPA2170_-IN_A_1: R16.1, U1.-IN_A
- new net OPA2170_-IN_B_1: R15.1, U1.-IN_B
- new net OPA2170_OUT_A_1: R16.2, R17.1, U1.OUT_A
- new net OPA2170_OUT_B_1: R15.2, R19.1, U1.OUT_B
- new net SYS5V_F: C3.C2, C8.C2, U1.V+, U6.V+, X1.A3
- net +3.3V: now also C12.C2, R28.1, R29.1, R30.1, R31.1, R32.1, R33.1, X1.A4; no longer C48.C2, R82.1, R83.1, R84.1, R85.1
- net 24AA_A1: now also R32.2, X2.4; no longer R84.2, U17.2
- net 24AA_WP: now also R30.2, X2.8; no longer R83.2, U17.1
- net AGND: now also C1.C1, C10.C1, C12.C1, C2.C1, C3.C1, C4.C1, C5.C1, C6.C1, C7.C1, C8.C1, C9.C1, R10.2, R13.1, R14.1, R18.2, R20.2, R3.1, R4.1, R8.2, U1.V-, U16.VSS, X1.B3, X1.B4, X2.1, X2.3, X2.5, X2.7; no longer C37.C1, C38.C1, C39.C1, C40.C1, C41.C1, R58.1, R59.1, R61.2, R63.2
- net AIN1_0-10V: now also R1.2, X1.A1; no longer C37.C2, R56.2
- net AIN2: now also C9.C2, R17.2, R18.1, X1.A8; no longer C39.C2, R60.2, R61.1
- net AIN2_0-10V: now also R2.2, X1.B1; no longer C38.C2, R57.2
- net AIN3: now also C10.C2, R19.2, R20.1, X1.B8; no longer C40.C2, R62.2, R63.1
- net I2C2_SCL: now also R29.2, X1.B6
- net I2C2_SDA: now also R28.2, X1.B5
- net N$21: now also C1.C2, R1.1, R3.2; no longer R56.1, R58.2
- net N$45: now also C2.C2, R2.1, R4.2; no longer R57.1, R59.2
- net OPA2170_-IN_A_2: now also R6.1; no longer R65.1
- net OPA2170_-IN_B_2: now also R5.1; no longer R64.1
- net OPA2170_OUT_A_2: now also R6.2, R7.1; no longer R60.1, R65.2
- net OPA2170_OUT_B_2: now also R5.2, R9.1; no longer R62.1, R64.2
Other:
- note added: "Set I2C slave address: b01010 A2 A1 A0"
- note removed: "I2C slave address: b1010100 = h54"
- note removed: "R56, R57: durch 9.76kOhm +/- 0.1% ersetzen R58, R59: durch 5.49kOhm +/- 0.1% ersetzen"
- note removed: "R60 - R63: durch 499 Ohm +/- 0.1% ersetzen"
- note removed: "mit 953 Ohm ersetzen"
- moved on the sheet: U16, U6
