File: EL-100-020-020-PT1000.sch (EAGLE design)
At the start: 46 parts, among them U1 OPA2188AIDGKR, U16 24AA256-I/SN, U2 OPA2188AIDGKR, U3 REF3025AIDBZTG4, U4 ADS1015IDGST, X1 944-12-2-00, X3 9012-26

Commit message: DIN rail PT1000 and indicator
Parts:
- removed C48: 0.1uF, Kemet_By_element14_Batch_1:C0603C104K5RAC-TU
- removed R82, R84, R85: 4.7K Ohms, Vishay_By_element14_Batch_1:CRCW06034K70FKEA
- removed R83: 10K Ohms, Vishay_By_element14_Batch_1:CRCW060310K0FKEA
- removed U3: REF3025AIDBZTG4, strasys_standard:REF3025AIDBZTG4
- added C1, C10, C4, C8, C9: 100nF, Kemet_By_element14_1:C0805C104K5RACTU
- added R30, R31, R32, R33: 10K Ohms, Vishay_By_element14_Batch_1:CRCW080510K0JNEA
- added REF1: LM4030CMF-2.5, strasys_standard:LM4030CMF-2.5
- added X2: 944-12-08-00, strasys_standard:944-12-08-00
- R1: value 10KOHM -> 10k Ohms; device Panasonic-Trimmer_Potentiometers:EVM3YSX50B14-3W -> Vishay_By_element14_Batch_1:CRCW080524K9FKEA; MF PANASONIC ELECTRONIC COMPONENTS -> (none); MPN (none) -> ERA6AEB103V; OC_FARNELL 1849801 -> 1577673; SUPPLIER (none) -> PANASONIC; TOLERANCE (none) -> ±0.1%
- R10: value 24.9K Ohms -> 10k Ohms; MF VISHAY DRALORIC -> (none); MPN (none) -> ERA6AEB103V; OC_FARNELL (none) -> 1577673; SUPPLIER (none) -> PANASONIC; TOLERANCE (none) -> ±0.1%
- R11: MF VISHAY DRALORIC -> (none); MPN (none) -> ERA6AEB102V; OC_FARNELL (none) -> 1577659; SUPPLIER (none) -> PANASONIC; TOLERANCE (none) -> ±0.1%
- R12, R6: MF VISHAY DRALORIC -> (none); MPN (none) -> MCTC0525B1053T5E; OC_FARNELL (none) -> 1576016; SUPPLIER (none) -> MULTICOMP; TOLERANCE (none) -> ±0.1%
- R13: value 10K Ohms -> 560 Ohms; MF VISHAY DRALORIC -> MULTICOMP; MPN (none) -> MCMR08X561 JTL; OC_FARNELL (none) -> 2073807; SUPPLIER (none) -> MULTICOMP
- R14, R20: value 10KOHM -> 12.7K Ohms; device Panasonic-Trimmer_Potentiometers:EVM3YSX50B14-3W -> Vishay_By_element14_Batch_1:CRCW080530K0FKEA; MF PANASONIC ELECTRONIC COMPONENTS -> (none); MPN (none) -> MCTC0525B1272T5E; OC_FARNELL 1849801 -> 1575914; SUPPLIER (none) -> MULTICOMP; TOLERANCE (none) -> ±0.1%
- R15, R21: value 30K Ohms -> 11.5kohms; device Vishay_By_element14_Batch_1:CRCW080530K0FKEA -> Vishay_By_element14_Batch_1:ERJ6ENF3242V; MF VISHAY DRALORIC -> (none); MPN (none) -> MCTC0525B1152T5E; OC_FARNELL (none) -> 1575906; SUPPLIER (none) -> MULTICOMP; TOLERANCE (none) -> +/- 0.1%
- R16, R22: value 32.4kohms -> 10k Ohms; device Vishay_By_element14_Batch_1:ERJ6ENF3242V -> Vishay_By_element14_Batch_1:CRCW080524K9FKEA; MF PANASONIC ELECTRONIC COMPONENTS -> (none); MPN (none) -> ERA6AEB103V; OC_FARNELL (none) -> 1577673; SUPPLIER (none) -> PANASONIC; TOLERANCE (none) -> ±0.1%
- R17, R23: value 24.9K Ohms -> 1K Ohms; device Vishay_By_element14_Batch_1:CRCW080524K9FKEA -> Vishay_By_element14_Batch_1:CRCW08051K00FKEA; MF VISHAY DRALORIC -> (none); MPN (none) -> ERA6AEB102V; OC_FARNELL (none) -> 1577659; SUPPLIER (none) -> PANASONIC; TOLERANCE (none) -> ±0.1%
- R18, R24: value 1K Ohms -> 105K Ohms; device Vishay_By_element14_Batch_1:CRCW08051K00FKEA -> Vishay_By_element14_Batch_1:CRCW0805105KFKEA; MF VISHAY DRALORIC -> (none); MPN (none) -> MCTC0525B1053T5E; OC_FARNELL (none) -> 1576016; SUPPLIER (none) -> MULTICOMP; TOLERANCE (none) -> ±0.1%
- R19, R25: value 105K Ohms -> 3K Ohms; device Vishay_By_element14_Batch_1:CRCW0805105KFKEA -> Vishay_By_element14_Batch_1:CRCW080530K0FKEA; MF VISHAY DRALORIC -> (none); MPN (none) -> ERA6AEB302V; OC_FARNELL (none) -> 1670234; SUPPLIER (none) -> Panasonic; TOLERANCE (none) -> ±0.1%
- R2: value 24.9K Ohms -> 11.5kohms; device Vishay_By_element14_Batch_1:CRCW080524K9FKEA -> Vishay_By_element14_Batch_1:ERJ6ENF3242V; MF VISHAY DRALORIC -> (none); MPN (none) -> MCTC0525B1152T5E; OC_FARNELL (none) -> 1575906; SUPPLIER (none) -> MULTICOMP; TOLERANCE (none) -> +/- 0.1%
- R3, R8: value 30K Ohms -> 12.7K Ohms; MF VISHAY DRALORIC -> (none); MPN (none) -> MCTC0525B1272T5E; OC_FARNELL (none) -> 1575914; SUPPLIER (none) -> MULTICOMP; TOLERANCE (none) -> ±0.1%
- R4: value 32.4kohms -> 1K Ohms; device Vishay_By_element14_Batch_1:ERJ6ENF3242V -> Vishay_By_element14_Batch_1:CRCW08051K00FKEA; MF PANASONIC ELECTRONIC COMPONENTS -> (none); MPN (none) -> ERA6AEB102V; OC_FARNELL (none) -> 1577659; SUPPLIER (none) -> PANASONIC; TOLERANCE (none) -> ±0.1%
- R5: value 1K Ohms -> 3K Ohms; device Vishay_By_element14_Batch_1:CRCW08051K00FKEA -> Vishay_By_element14_Batch_1:CRCW080530K0FKEA; MF VISHAY DRALORIC -> (none); MPN (none) -> ERA6AEB302V; OC_FARNELL (none) -> 1670234; SUPPLIER (none) -> Panasonic; TOLERANCE (none) -> ±0.1%
- R7: value 10KOHM -> 3K Ohms; device Panasonic-Trimmer_Potentiometers:EVM3YSX50B14-3W -> Vishay_By_element14_Batch_1:CRCW080530K0FKEA; MF PANASONIC ELECTRONIC COMPONENTS -> (none); MPN (none) -> ERA6AEB302V; OC_FARNELL 1849801 -> 1670234; SUPPLIER (none) -> Panasonic; TOLERANCE (none) -> ±0.1%
- R9: value 32.4kohms -> 11.5kohms; MF PANASONIC ELECTRONIC COMPONENTS -> (none); MPN (none) -> MCTC0525B1152T5E; OC_FARNELL (none) -> 1575906; SUPPLIER (none) -> MULTICOMP; TOLERANCE (none) -> +/- 0.1%
- X1: value 944-12-2-00 -> 944-12-08-00; device strasys_standard:944-12-2-00 -> strasys_standard:944-12-08-00
Connections:
- net I2C2_SDA renamed N$4
- removed net +3.3V1: R28.1, R29.1
- removed net 24AA_A0: R85.2, U16.A0
- removed net DGND: C48.C1, U16.VSS, X1.1
- removed net N$19: R82.2, U16.A2
- removed net N$2: R14.1, R15.1
- removed net N$3: R7.1, R8.1
- removed net N$4 (its old number): R20.1, R21.1
- removed net N$6: R1.1, R3.1
- removed net P9_14: R13.2, U4.ALERT/RDY
- new net +IN_0: C4.C2, R5.1, R6.2, U1.+IN_A
- new net +IN_1: C1.C2, R12.2, R7.1, U1.+IN_B
- new net +IN_2: C8.C2, R18.2, R19.1, U2.+IN_A
- new net +IN_3: C9.C2, R24.2, R25.1, U2.+IN_B
- new net 24AA-A0: R31.2, U16.A0, X2.2
- new net 24AA_A2: R33.2, U16.A2, X2.6
- new net ADDR: U4.ADDR, X1.1, X1.3, X1.5, X1.7
- new net N$1: R13.1, REF1.-GND
- net +3.3V: now also C10.C2, R28.1, R29.1, R30.1, R31.1, R32.1, R33.1; no longer C48.C2, R13.1, R82.1, R83.1, R84.1, R85.1
- net -IN_0: now also R2.1; no longer R5.1
- net -IN_2: now also R14.2, R15.1, R17.1; no longer R15.2, R16.1, R18.1
- net -IN_3: now also R20.2, R21.1, R23.1; no longer R21.2, R22.1, R24.1
- net 24AA_A1: now also R32.2, X2.4; no longer R84.2
- net 24AA_WP: now also R30.2, X2.8; no longer R83.2, X1.2
- net AGND: now also C1.C1, C10.C1, C4.C1, C8.C1, C9.C1, R17.2, R23.2, R4.2, REF1.GND, U16.VSS, U4.ALERT/RDY, X1.2, X2.1, X2.3, X2.5, X2.7; no longer R18.2, R24.2, R5.2, U3.GND, U4.ADDR
- net AIN0: now also R3.1; no longer R1.2
- net AIN1: now also R8.1; no longer R7.2
- net AIN2: now also R14.1, R18.1; no longer R14.2, R19.1
- net AIN3: now also R20.1, R24.1; no longer R20.2, R25.1
- net I2C1_SCL: now also X1.8
- net I2C1_SDA: now also X1.6
- net PT1000_0: now also R1.2, R5.2; no longer R2.2, R6.2, U1.+IN_A
- net PT1000_1: now also R7.2; no longer R12.2, U1.+IN_B
- net PT1000_2: now also R16.2; no longer R17.2, U2.+IN_A
- net PT1000_3: now also R22.2; no longer R23.2, U2.+IN_B
- net REF2.5V: now also R1.1, R15.2, R16.1, R2.2, R21.2, R22.1, REF1.+VREF; no longer R16.2, R17.1, R2.1, R22.2, R23.1, R4.2, U3.OUT
- net SYS5V_F: now also R13.2, X1.4; no longer U3.IN
Other:
- note added: "1001000 (0x48) ADDR PIN => GND 1001001 (0x49) ADDR PIN => VDD 1001010 (0x4A) ADDR PIN => SDA 1001011 (0x4B) ADDR PIN => SCL"
- note added: "Ersetzen durch LM4030B"
- note added: "Set I2C slave address: b01010 A2 A1 A0"
- note removed: "I2C address: 1001000 (h48) ADDR to GND"
- note removed: "I2C slave address: b1010100 = h54"

Commit message: prototype order status
Connections:
- net N$4 renamed I2C2_SDA
Changed lines of the file:
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@@
-</segment>
-</net>
-<net name="N$4" class="0">
-<segment>
-<pinref part="U16" gate="A" pin="SDA"/>
-<wire x1="152.4" y1="73.66" x2="182.88" y2="73.66" width="0.1524" layer="91"/>
-<label x="185.42" y="73.66" size="1.778" layer="95"/>
-</segment>
-<segment>
-<wire x1="259.08" y1="43.18" x2="220.98" y2="43.18" width="0.1524" layer="91"/>
-<wire x1="220.98" y1="43.18" x2="213.36" y2="43.18" width="0.1524" layer="91"/>
-<wire x1="220.98" y1="55.88" x2="220.98" y2="43.18" width="0.1524" layer="91"/>
-<junction x="220.98" y="43.18"/>
-<label x="261.62" y="43.18" size="1.778" layer="95"/>
-<pinref part="R28" gate="A" pin="2"/>
-</segment>
-<segment>
-<pinref part="X3" gate="G$1" pin="B5"/>
-<wire x1="167.64" y1="190.5" x2="172.72" y2="190.5" width="0.1524" layer="91"/>
-<label x="175.26" y="190.5" size="1.778" layer="95"/>
 </segment>
 </net>
@@
 </segment>
 </net>
+<net name="I2C2_SDA" class="0">
+<segment>
+<wire x1="259.08" y1="43.18" x2="220.98" y2="43.18" width="0.1524" layer="91"/>
+<wire x1="220.98" y1="43.18" x2="213.36" y2="43.18" width="0.1524" layer="91"/>
+<wire x1="220.98" y1="55.88" x2="220.98" y2="43.18" width="0.1524" layer="91"/>
+<junction x="220.98" y="43.18"/>
+<label x="261.62" y="43.18" size="1.778" layer="95"/>
+<pinref part="R28" gate="A" pin="2"/>
+</segment>
+<segment>
+<pinref part="U16" gate="A" pin="SDA"/>
+<wire x1="152.4" y1="73.66" x2="182.88" y2="73.66" width="0.1524" layer="91"/>
+<label x="185.42" y="73.66" size="1.778" layer="95"/>
+</segment>
+<segment>
+<pinref part="X3" gate="G$1" pin="B5"/>
+<wire x1="167.64" y1="190.5" x2="172.72" y2="190.5" width="0.1524" layer="91"/>
+<label x="175.26" y="190.5" size="1.778" layer="95"/>
+</segment>
+</net>
