File: EL-100-020-005-indicator-light.brd (EAGLE design)
At the start: 20 x 39.8 mm, 13 parts, among them X1 140-08-FLACHBAND1.27

Commit message: prototype order status
Parts:
- LED4: value KP-1608QBC-D-LED -> P-1608SURCK
Changed lines of the file:
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@@
 <attribute name="VALUE" x="3.2" y="14.9" size="1.778" layer="27"/>
 </element>
-<element name="LED4" library="strasys_standard" package="KP-1608QBCD-D-LED" value="KP-1608QBC-D-LED" x="5" y="12.4" smashed="yes">
+<element name="LED4" library="strasys_standard" package="KP-1608QBCD-D-LED" value="P-1608SURCK" x="5" y="12.4" smashed="yes">
 <attribute name="SUPPLIER" value="Kingbright" x="5" y="12.4" size="1.778" layer="27" display="off"/>
-<attribute name="MPC" value="KP-1608QBC-D-LED" x="5" y="12.4" size="1.778" layer="27" display="off"/>
-<attribute name="OC_FARNELL" value="2217972" x="5" y="12.4" size="1.778" layer="27" display="off"/>
+<attribute name="MPC" value="KP-1608SURCK" x="5" y="12.4" size="1.778" layer="27" display="off"/>
+<attribute name="OC_FARNELL" value="2290329" x="5" y="12.4" size="1.778" layer="27" display="off"/>
 <attribute name="NAME" x="3.8" y="10.4" size="1.016" layer="25"/>
 <attribute name="VALUE" x="3.2" y="9.9" size="1.778" layer="27"/>
