File: EL-100-020-020-PT1000.brd (EAGLE design)
At the start: 54 x 29.5 mm, 53 parts, among them U1 OPA2188AIDGKR, U16 24AA256-I/SN, U2 OPA2188AIDGKR, U4 ADS1015IDGST, X1 944-12-08-00, X2 944-12-08-00, X3 9012-26

Commit message: prototype order status
Connections:
- net N$4 renamed I2C2_SDA
Changed lines of the file:
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@@
 <layer number="16" name="Bottom" color="1" fill="1" visible="yes" active="yes"/>
 <layer number="17" name="Pads" color="2" fill="1" visible="yes" active="yes"/>
-<layer number="18" name="Vias" color="2" fill="1" visible="yes" active="yes"/>
-<layer number="19" name="Unrouted" color="6" fill="1" visible="yes" active="yes"/>
+<layer number="18" name="Vias" color="2" fill="1" visible="no" active="yes"/>
+<layer number="19" name="Unrouted" color="6" fill="1" visible="no" active="yes"/>
 <layer number="20" name="Dimension" color="15" fill="1" visible="yes" active="yes"/>
 <layer number="21" name="tPlace" color="7" fill="1" visible="yes" active="yes"/>
-<layer number="22" name="bPlace" color="7" fill="1" visible="yes" active="yes"/>
+<layer number="22" name="bPlace" color="7" fill="1" visible="no" active="yes"/>
 <layer number="23" name="tOrigins" color="15" fill="1" visible="yes" active="yes"/>
-<layer number="24" name="bOrigins" color="15" fill="1" visible="yes" active="yes"/>
+<layer number="24" name="bOrigins" color="15" fill="1" visible="no" active="yes"/>
 <layer number="25" name="tNames" color="7" fill="1" visible="yes" active="yes"/>
-<layer number="26" name="bNames" color="7" fill="1" visible="yes" active="yes"/>
+<layer number="26" name="bNames" color="7" fill="1" visible="no" active="yes"/>
 <layer number="27" name="tValues" color="7" fill="1" visible="no" active="yes"/>
 <layer number="28" name="bValues" color="7" fill="1" visible="no" active="yes"/>
@@
 <layer number="37" name="tTest" color="7" fill="1" visible="no" active="yes"/>
 <layer number="38" name="bTest" color="7" fill="1" visible="no" active="yes"/>
-<layer number="39" name="tKeepout" color="4" fill="11" visible="yes" active="yes"/>
-<layer number="40" name="bKeepout" color="1" fill="11" visible="yes" active="yes"/>
-<layer number="41" name="tRestrict" color="4" fill="10" visible="yes" active="yes"/>
-<layer number="42" name="bRestrict" color="1" fill="10" visible="yes" active="yes"/>
-<layer number="43" name="vRestrict" color="2" fill="10" visible="yes" active="yes"/>
+<layer number="39" name="tKeepout" color="4" fill="11" visible="no" active="yes"/>
+<layer number="40" name="bKeepout" color="1" fill="11" visible="no" active="yes"/>
+<layer number="41" name="tRestrict" color="4" fill="10" visible="no" active="yes"/>
+<layer number="42" name="bRestrict" color="1" fill="10" visible="no" active="yes"/>
+<layer number="43" name="vRestrict" color="2" fill="10" visible="no" active="yes"/>
 <layer number="44" name="Drills" color="7" fill="1" visible="no" active="yes"/>
 <layer number="45" name="Holes" color="7" fill="1" visible="no" active="yes"/>
 <layer number="46" name="Milling" color="3" fill="1" visible="no" active="yes"/>
 <layer number="47" name="Measures" color="7" fill="1" visible="yes" active="yes"/>
-<layer number="48" name="Document" color="7" fill="1" visible="yes" active="yes"/>
-<layer number="49" name="Reference" color="7" fill="1" visible="yes" active="yes"/>
+<layer number="48" name="Document" color="7" fill="1" visible="no" active="yes"/>
+<layer number="49" name="Reference" color="7" fill="1" visible="no" active="yes"/>
 <layer number="50" name="dxf" color="7" fill="1" visible="no" active="no"/>
 <layer number="51" name="tDocu" color="7" fill="1" visible="no" active="yes"/>
-<layer number="52" name="bDocu" color="7" fill="1" visible="yes" active="yes"/>
+<layer number="52" name="bDocu" color="7" fill="1" visible="no" active="yes"/>
 <layer number="53" name="tPadExt" color="7" fill="1" visible="no" active="no"/>
 <layer number="54" name="bPadExt" color="7" fill="1" visible="no" active="no"/>
@@
 <layer number="97" name="Info" color="7" fill="1" visible="no" active="no"/>
 <layer number="98" name="Guide" color="6" fill="1" visible="no" active="no"/>
-<layer number="250" name="Descript" color="7" fill="1" visible="yes" active="yes"/>
-<layer number="251" name="SMDround" color="7" fill="1" visible="yes" active="yes"/>
+<layer number="250" name="Descript" color="7" fill="1" visible="no" active="yes"/>
+<layer number="251" name="SMDround" color="7" fill="1" visible="no" active="yes"/>
 </layers>
 <board>
@@
 <text x="3.8" y="24.8" size="1" layer="1" font="vector" ratio="15">PT1000</text>
 <text x="9" y="24.8" size="1" layer="16" font="vector" ratio="15" rot="MR0">PT1000</text>
-<dimension x1="0" y1="0" x2="0" y2="29.5" x3="-3.4" y3="14.75" textsize="1.778" layer="47"/>
-<dimension x1="0" y1="0" x2="54" y2="0" x3="27" y3="-3.6" textsize="1.778" layer="47" dtype="horizontal"/>
+<dimension x1="0" y1="0" x2="0" y2="29.5" x3="-3.4" y3="14.75" textsize="1" textratio="15" layer="47"/>
+<dimension x1="0" y1="0" x2="54" y2="0" x3="27" y3="-3.2" textsize="1" textratio="15" layer="47" dtype="horizontal"/>
 </plain>
 <attributes>
@@
 <attribute name="MF" value="MICROCHIP" x="12.3" y="102.4" size="1.778" layer="27" rot="R90" display="off"/>
 <attribute name="OC_FARNELL" value="1331295" x="12.3" y="102.4" size="1.778" layer="27" rot="R90" display="off"/>
-<attribute name="NAME" x="9.4456" y="20.2412" size="1.016" layer="25" font="vector" rot="SR270"/>
+<attribute name="NAME" x="2.0544" y="15.8588" size="1.016" layer="25" font="vector" rot="SR90"/>
 <attribute name="VALUE" x="10.8522" y="13.0174" size="2.0828" layer="27" ratio="10" rot="SR90"/>
 </element>
@@
 <signal name="N$2">
 </signal>
-<signal name="N$4">
-<wire x1="7.8" y1="19.5" x2="7.8" y2="19.2" width="0.2" layer="16"/>
-<wire x1="7.8" y1="19.2" x2="7.5" y2="18.9" width="0.2" layer="16"/>
-<wire x1="7.5" y1="18.9" x2="7.2" y2="18.9" width="0.2" layer="16"/>
-<wire x1="7.2" y1="18.9" x2="7" y2="18.7" width="0.2" layer="16"/>
-<wire x1="7" y1="18.7" x2="7" y2="15.6" width="0.2" layer="16"/>
-<wire x1="7" y1="15.6" x2="13" y2="9.6" width="0.2" layer="16"/>
-<contactref element="U16" pad="5"/>
-<contactref element="R28" pad="2"/>
-<contactref element="X3" pad="B5"/>
-<wire x1="14.2" y1="9.6" x2="14.2" y2="7.8" width="0.2" layer="1"/>
-<wire x1="23.6" y1="9.6" x2="14.2" y2="9.6" width="0.2" layer="16"/>
-<wire x1="24.2" y1="10.2" x2="23.6" y2="9.6" width="0.2" layer="16"/>
-<wire x1="24.2" y1="9.4" x2="24.2" y2="10.2" width="0.2" layer="1"/>
-<wire x1="24.4" y1="9.2" x2="24.2" y2="9.4" width="0.2" layer="1"/>
-<wire x1="14.2" y1="7.8" x2="14.2398" y2="7.8" width="0.2" layer="1"/>
-<wire x1="24.4" y1="9.2" x2="24.45" y2="9.28" width="0.2" layer="1"/>
-<via x="14.2" y="9.6" extent="1-16" drill="0.3"/>
-<via x="24.2" y="10.2" extent="1-16" drill="0.3"/>
-<via x="7.8" y="19.5" extent="1-16" drill="0.3"/>
-<wire x1="7.9" y1="19.6" x2="7.8" y2="19.5" width="0.2" layer="1"/>
-<wire x1="7.9" y1="20.9" x2="7.9" y2="19.6" width="0.2" layer="1"/>
-<wire x1="7.9" y1="20.9" x2="7.855" y2="20.9422" width="0.2" layer="1"/>
-<wire x1="13" y1="9.6" x2="14.2" y2="9.6" width="0.2" layer="16"/>
-</signal>
 <signal name="PE">
 <polygon width="0.2" layer="1" rank="6">
@@
 </polygon>
 </signal>
+<signal name="I2C2_SDA">
+<contactref element="R28" pad="2"/>
+<contactref element="U16" pad="5"/>
+<wire x1="7.8" y1="19.5" x2="7.8" y2="19.2" width="0.2" layer="16"/>
+<wire x1="7.8" y1="19.2" x2="7.5" y2="18.9" width="0.2" layer="16"/>
+<wire x1="7.5" y1="18.9" x2="7.2" y2="18.9" width="0.2" layer="16"/>
+<wire x1="7.2" y1="18.9" x2="7" y2="18.7" width="0.2" layer="16"/>
+<wire x1="7" y1="18.7" x2="7" y2="15.6" width="0.2" layer="16"/>
+<wire x1="7" y1="15.6" x2="13" y2="9.6" width="0.2" layer="16"/>
+<contactref element="X3" pad="B5"/>
+<wire x1="14.2" y1="9.6" x2="14.2" y2="7.8" width="0.2" layer="1"/>
+<wire x1="23.6" y1="9.6" x2="14.2" y2="9.6" width="0.2" layer="16"/>
+<wire x1="24.2" y1="10.2" x2="23.6" y2="9.6" width="0.2" layer="16"/>
+<wire x1="24.2" y1="9.4" x2="24.2" y2="10.2" width="0.2" layer="1"/>
+<wire x1="24.4" y1="9.2" x2="24.2" y2="9.4" width="0.2" layer="1"/>
+<wire x1="24.4" y1="9.2" x2="24.45" y2="9.28" width="0.2" layer="1"/>
+<via x="14.2" y="9.6" extent="1-16" drill="0.3"/>
+<via x="24.2" y="10.2" extent="1-16" drill="0.3"/>
+<via x="7.8" y="19.5" extent="1-16" drill="0.3"/>
+<wire x1="7.9" y1="19.6" x2="7.8" y2="19.5" width="0.2" layer="1"/>
+<wire x1="7.9" y1="20.9" x2="7.9" y2="19.6" width="0.2" layer="1"/>
+<wire x1="13" y1="9.6" x2="14.2" y2="9.6" width="0.2" layer="16"/>
+<wire x1="7.9" y1="20.9" x2="7.855" y2="20.9422" width="0" layer="19" extent="1-1"/>
+<wire x1="14.2398" y1="7.8" x2="14.2" y2="7.8" width="0" layer="19" extent="1-1"/>
+</signal>
 </signals>
